Commit message: [update] package updated by sayna

File: dsr_description/xacro/m0609.urdf.xacro (robot description, xacro)
@@ -11,5 +11,5 @@
      <xacro:include filename="$(find dsr_description)/xacro/macro.m0609.blue.xacro" />
   </xacro:if>
-  <xacro:m0609 namespace="$(arg namespace)"/>
+  <xacro:m0609 namespace="dsr01m0609"/>
   <link name="world" />
   <xacro:if value="${gr == 'robotiq_2f'}">

File: dsr_description/xacro/robotiq_2f.urdf.xacro (robot description, xacro)
@@ -33,10 +33,10 @@
   </gazebo>
   <!-- Equivalent to the OpenRAVE manipulator denso_robotiq_85_gripper -->
-  <!-- <link name="denso_robotiq_85_gripper" /> -->
-  <!-- <joint name="manipulator_dummy_joint" type="fixed"> -->
-  <!--   <origin xyz="0 0 0.1441" rpy="0 0 0" /> -->
-  <!--   <parent link="robotiq_coupler"/> -->
-  <!--   <child link="denso_robotiq_85_gripper"/> -->
-  <!-- </joint> -->
+  <link name="denso_robotiq_85_gripper" />
+  <joint name="manipulator_dummy_joint" type="fixed">
+    <origin xyz="0 0 0.1441" rpy="0 0 0" />
+    <parent link="robotiq_coupler"/>
+    <child link="denso_robotiq_85_gripper"/>
+  </joint>
   <!-- Attach the robotiq 85 gripper -->
   <xacro:robotiq_85_gripper prefix="" parent="robotiq_coupler" >
